Commit message: feat(ec66): 添加ikfast插件

File: src/elite_description/urdf/ec66_description.urdf (robot description, URDF)
Before this commit: robot ec66, 9 links, 8 joints
Links:
- link flan: mass None -> 0.10466; geometry collision box size=0 0 0; visual box size=0 0 0
Joints:
- joint flan_joint: axis (none) -> 0 0 0; origin xyz=0 0 0 rpy=0 0 0 -> xyz=0 -0.089 -0.00047661 rpy=-1.5708 0 3.1416
- joint joint1: limit lower=-6.2832 upper=6.2832 effort=150.0 velocity=2.61993 -> lower=-6.2832 upper=6.2832 effort=150 velocity=2.6199; origin xyz=0 0 0.096 rpy=0 0 3.1416 -> xyz=0 0 0.096 rpy=0 0 0
- joint joint2: axis 0 0 1 -> 0 1 0; limit lower=-6.2832 upper=6.2832 effort=150.0 velocity=2.61993 -> lower=-6.2832 upper=6.2832 effort=150 velocity=2.6199; origin xyz=0 0 0 rpy=1.5708 -1.5708 0 -> xyz=0 0.122 0 rpy=0 1.5708 0
- joint joint3: axis 0 0 1 -> 0 1 0; limit lower=-2.7925 upper=2.7925 effort=150.0 velocity=3.31613 -> lower=-2.7925 upper=2.7925 effort=150 velocity=3.3161; origin xyz=0 0.418 0 rpy=0 0 1.5708 -> xyz=0 -0.122 0.418 rpy=0 0 0
- joint joint4: axis 0 0 1 -> 0 1 0; limit lower=-6.2832 upper=6.2832 effort=28.0 velocity=4.53786 -> lower=-6.2832 upper=6.2832 effort=28 velocity=4.5379; origin xyz=0.398 0 0.122 rpy=0 0 0 -> xyz=0 0 0.398 rpy=0 1.5708 0
- joint joint5: limit lower=-6.2832 upper=6.2832 effort=28.0 velocity=4.53786 -> lower=-6.2832 upper=6.2832 effort=28 velocity=4.5379; origin xyz=0 0.098 0 rpy=1.5708 0 -3.1416 -> xyz=0 0.122 0 rpy=0 0 0
- joint joint6: axis 0 0 1 -> 0 -1 0; limit lower=-6.2832 upper=6.2832 effort=28.0 velocity=4.53786 -> lower=-6.2832 upper=6.2832 effort=28 velocity=4.5379; origin xyz=0 -0.089 0 rpy=-1.5708 0 3.1416 -> xyz=0 0 0.098 rpy=0 0 0

File: src/elite_description/urdf/gazebo/ec66_description.urdf (robot description, URDF)
Before this commit: robot ec66, 9 links, 8 joints
Links:
- link flan: mass None -> 0.10466; geometry collision box size=0 0 0; visual box size=0 0 0
Joints:
- joint flan_joint: axis (none) -> 0 0 0; origin xyz=0 0 0 rpy=0 0 0 -> xyz=0 -0.089 -0.00047661 rpy=-1.5708 0 3.1416
- joint joint1: limit lower=-6.2832 upper=6.2832 effort=150.0 velocity=2.61993 -> lower=-6.2832 upper=6.2832 effort=150 velocity=2.6199; origin xyz=0 0 0.096 rpy=0 0 3.1416 -> xyz=0 0 0.096 rpy=0 0 0
- joint joint2: axis 0 0 1 -> 0 1 0; limit lower=-6.2832 upper=6.2832 effort=150.0 velocity=2.61993 -> lower=-6.2832 upper=6.2832 effort=150 velocity=2.6199; origin xyz=0 0 0 rpy=1.5708 -1.5708 0 -> xyz=0 0.122 0 rpy=0 1.5708 0
- joint joint3: axis 0 0 1 -> 0 1 0; limit lower=-2.7925 upper=2.7925 effort=150.0 velocity=3.31613 -> lower=-2.7925 upper=2.7925 effort=150 velocity=3.3161; origin xyz=0 0.418 0 rpy=0 0 1.5708 -> xyz=0 -0.122 0.418 rpy=0 0 0
- joint joint4: axis 0 0 1 -> 0 1 0; limit lower=-6.2832 upper=6.2832 effort=28.0 velocity=4.53786 -> lower=-6.2832 upper=6.2832 effort=28 velocity=4.5379; origin xyz=0.398 0 0.122 rpy=0 0 0 -> xyz=0 0 0.398 rpy=0 1.5708 0
- joint joint5: limit lower=-6.2832 upper=6.2832 effort=28.0 velocity=4.53786 -> lower=-6.2832 upper=6.2832 effort=28 velocity=4.5379; origin xyz=0 0.098 0 rpy=1.5708 0 -3.1416 -> xyz=0 0.122 0 rpy=0 0 0
- joint joint6: axis 0 0 1 -> 0 -1 0; limit lower=-6.2832 upper=6.2832 effort=28.0 velocity=4.53786 -> lower=-6.2832 upper=6.2832 effort=28 velocity=4.5379; origin xyz=0 -0.089 0 rpy=-1.5708 0 3.1416 -> xyz=0 0 0.098 rpy=0 0 0
